File: Balance_LED/ESP32_H2.kicad_sch (KiCad schematic)
At the start: 0 parts

Commit message: Closed kicad
Parts:
- added J1: USB_C_Receptacle_USB2.0_16P, Connector_USB:USB_C_Receptacle_HCTL_HC-TYPE-C-16P-01A, symbol Connector:USB_C_Receptacle_USB2.0_16P
- added U1: ESP32-H2-MINI-1-H2, ESP32-H2-MINI-1-H2:MODULE_ESP32-H2-MINI-1-H2, symbol ESP32-H2-MINI-1-H2:ESP32-H2-MINI-1-H2
Connections:
- new net: U1.1 (GND_1), U1.11 (GND_1), U1.14 (GND_1), U1.2 (GND_1), U1.36 (GND_1), U1.37 (GND_1), U1.38 (GND_1), U1.39 (GND_1), U1.40 (GND_1), U1.41 (GND_1), U1.42 (GND_1), U1.43 (GND_1), U1.44 (GND_1), U1.45 (GND_1), U1.46 (GND_1)
- new net: U1.17 (NC), U1.28 (NC), U1.29 (NC), U1.32 (NC), U1.33 (NC), U1.34 (NC), U1.35 (NC), U1.4 (NC), U1.7 (NC)
- new net: U1.47 (GND_2), U1.48 (GND_2), U1.49_1 (GND_2), U1.49_2 (GND_2), U1.49_3 (GND_2), U1.49_4 (GND_2), U1.49_5 (GND_2), U1.49_6 (GND_2), U1.49_7 (GND_2), U1.49_8 (GND_2), U1.49_9 (GND_2), U1.50 (GND_2), U1.51 (GND_2), U1.52 (GND_2), U1.53 (GND_2)
- new net: J1.A4 (VBUS), J1.A9 (VBUS), J1.B4 (VBUS), J1.B9 (VBUS)
- new net GND: J1.A1 (GND), J1.A12 (GND), J1.B1 (GND), J1.B12 (GND), J1.S1 (SHIELD)
